File: design/Labor Oszi.kicad_sch (KiCad schematic)
At the start: 23 parts, among them J4 Conn_Coaxial, SW1 SW_SPDT, SW2 SW_SPDT, U1 NUCLEO-L432KC, U2 MCP6002-xMC, U3 MCP6002-xMC

Commit message: Schaltplan Revision
Parts:
- C1, C2: LCSC Part # (none) -> C14663
- R1: LCSC Part # (none) -> C23146
- R10: LCSC Part # (none) -> C23265
- R11, R5: LCSC Part # (none) -> C22961
- R12, R6: LCSC Part # (none) -> C23137
- R13: LCSC Part # (none) -> C4184
- R14: LCSC Part # (none) -> C23260
- R2, R4, R8: LCSC Part # (none) -> C25822
- R3: LCSC Part # (none) -> C22107
- R7: LCSC Part # (none) -> C23263
- R9: LCSC Part # (none) -> C23254
- U2, U3: LCSC Part # (none) -> C7377
Other:
- title: (none) -> Oszilloskop
Changed lines of the file:
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@@
 	(generator_version "9.0")
 	(paper "A4")
+	(title_block
+		(title "Oszilloskop")
+		(rev "Version 1.0")
+	)
 	(junction
 		(at 248.92 44.45)
@@
 			)
 		)
+		(property "LCSC Part #" "C25822"
+			(at 171.45 90.17 90)
+			(effects
+				(font
+					(size 1.27 1.27)
+				)
+				(hide yes)
+			)
+		)
 		(pin "1"
 		)
@@
 			)
 		)
+		(property "LCSC Part #" "C22961"
+			(at 121.92 81.28 0)
+			(effects
+				(font
+					(size 1.27 1.27)
+				)
+				(hide yes)
+			)
+		)
 		(pin "2"
 		)
@@
 			)
 		)
+		(property "LCSC Part #" "C23254"
+			(at 181.61 34.29 0)
+			(effects
+				(font
+					(size 1.27 1.27)
+				)
+				(hide yes)
+			)
+		)
 		(pin "2"
 		)
@@
 			)
 		)
+		(property "LCSC Part #" "C23146"
+			(at 111.76 43.18 90)
+			(effects
+				(font
+					(size 1.27 1.27)
+				)
+				(hide yes)
+			)
+		)
 		(pin "1"
 		)
@@
 			)
 		)
+		(property "LCSC Part #" "C7377"
+			(at 234.95 33.02 0)
+			(effects
+				(font
+					(size 1.27 1.27)
+				)
+				(hide yes)
+			)
+		)
 		(pin "2"
 		)
@@
 			)
 		)
+		(property "LCSC Part #" "C7377"
+			(at 236.22 67.31 0)
+			(effects
+				(font
+					(size 1.27 1.27)
+				)
+				(hide yes)
+			)
+		)
 		(pin "2"
 		)
@@
 			)
 		)
+		(property "LCSC Part #" "C4184"
+			(at 248.92 38.1 0)
+			(effects
+				(font
+					(size 1.27 1.27)
+				)
+				(hide yes)
+			)
+		)
 		(pin "1"
 		)
@@
 			)
 		)
+		(property "LCSC Part #" "C23137"
+			(at 121.92 99.06 0)
+			(effects
+				(font
+					(size 1.27 1.27)
+				)
+				(hide yes)
+			)
+		)
 		(pin "2"
 		)
@@
 			)
 		)
+		(property "LCSC Part #" "C23137"
+			(at 181.61 99.06 0)
+			(effects
+				(font
+					(size 1.27 1.27)
+				)
+				(hide yes)
+			)
+		)
 		(pin "2"
 		)
@@
 			)
 		)
+		(property "LCSC Part #" "C7377"
+			(at 234.95 95.25 0)
+			(effects
+				(font
+					(size 1.27 1.27)
+				)
+				(hide yes)
+			)
+		)
 		(pin "2"
 		)
@@
 			)
 		)
+		(property "LCSC Part #" "C25822"
+			(at 111.76 90.17 90)
+			(effects
+				(font
+					(size 1.27 1.27)
+				)
+				(hide yes)
+			)
+		)
 		(pin "1"
 		)
@@
 			)
 		)
+		(property "LCSC Part #" "C22107"
+			(at 121.92 34.29 0)
+			(effects
+				(font
+					(size 1.27 1.27)
+				)
+				(hide yes)
+			)
+		)
 		(pin "2"
 		)
@@
 			)
 		)
+		(property "LCSC Part #" "C23260"
+			(at 248.92 49.53 0)
+			(effects
+				(font
+					(size 1.27 1.27)
+				)
+				(hide yes)
+			)
+		)
 		(pin "1"
 		)
@@
 			)
 		)
+		(property "LCSC Part #" "C7377"
+			(at 236.22 127 0)
+			(effects
+				(font
+					(size 1.27 1.27)
+				)
+				(hide yes)
+			)
+		)
 		(pin "2"
 		)
@@
 			)
 		)
+		(property "LCSC Part #" "C23263"
+			(at 171.45 43.18 90)
+			(effects
+				(font
+					(size 1.27 1.27)
+				)
+				(hide yes)
+			)
+		)
 		(pin "1"
 		)
@@
 			)
 		)
+		(property "LCSC Part #" "C23265"
+			(at 181.61 52.07 0)
+			(effects
+				(font
+					(size 1.27 1.27)
+				)
+				(hide yes)
+			)
+		)
 		(pin "2"
 		)
@@
 			)
 		)
+		(property "LCSC Part #" "C14663"
+			(at 214.63 50.8 0)
+			(effects
+				(font
+					(size 1.27 1.27)
+				)
+				(hide yes)
+			)
+		)
 		(pin "1"
 		)
@@
 			)
 		)
+		(property "LCSC Part #" "C22961"
+			(at 181.61 81.28 0)
+			(effects
+				(font
+					(size 1.27 1.27)
+				)
+				(hide yes)
+			)
+		)
 		(pin "2"
 		)
@@
 			)
 		)
+		(property "LCSC Part #" "C25822"
+			(at 121.92 52.07 0)
+			(effects
+				(font
+					(size 1.27 1.27)
+				)
+				(hide yes)
+			)
+		)
 		(pin "2"
 		)
@@
 			(at 207.01 113.03 0)
 			(effects
+				(font
+					(size 1.27 1.27)
+				)
+				(hide yes)
+			)
+		)
+		(property "LCSC Part #" "C14663"
+			(at 207.01 113.03 0)
+			(effects

Commit message: minor Part changes & Folder Structure fixes
Parts:
- U2, U3: LCSC Part # C7377 -> C185041
Changed lines of the file:
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@@
 	(title_block
 		(title "Oszilloskop")
-		(rev "Version 1.0")
+		(rev "Version 1.1")
 	)
 	(junction
@@
 			)
 		)
-		(property "LCSC Part #" "C7377"
+		(property "LCSC Part #" "C185041"
 			(at 234.95 33.02 0)
 			(effects
@@
 			)
 		)
-		(property "LCSC Part #" "C7377"
+		(property "LCSC Part #" "C185041"
 			(at 236.22 67.31 0)
 			(effects
@@
 			)
 		)
-		(property "LCSC Part #" "C7377"
+		(property "LCSC Part #" "C185041"
 			(at 234.95 95.25 0)
 			(effects
@@
 			)
 		)
-		(property "LCSC Part #" "C7377"
+		(property "LCSC Part #" "C185041"
 			(at 236.22 127 0)
 			(effects
