File: design/Labor Oszi.kicad_pcb (KiCad board)
At the start: 2 copper layers, 64.4 x 40.4 mm, 23 parts, among them J4 Conn_Coaxial, SW1 SW_SPDT, SW2 SW_SPDT, U1 NUCLEO-L432KC, U2 MCP6002-xMC, U3 MCP6002-xMC

Commit message: minor changes on the pcb
Parts:
- moved U1 11.0 mm to (156.4, 76.8), turned to -90 degrees
Routing:
- net /CH1_OPV2: track 52.1 -> 21.7 mm
- net /CH1_OPV1: track 43.4 -> 21.8 mm, vias 4 -> 2
- net /3.3V: track 90.8 -> 77.5 mm
- net /CH0_OPV1: track 52.3 -> 48.1 mm
- net /CH0_OPV2: track 33.0 -> 34.8 mm
Other:
- board text added: "Version 1.1 Made by Sonja Schönauer & Nicolas Scherrer"
